Commit message: 修正701路线、自旋跟踪与Gazebo仿真，移除导航停止接口

File: src/sentry_sim/robots/sentry.urdf (robot description, URDF)
Before this commit: robot sentry_simulator, 1 links, 0 joints
Links:
- removed link vehicle
- added link front_left_wheel, mass 0.4; collision cylinder length=0.0452 radius=0.0758; visual mesh filename=model://sentry_robot_visual/meshes/wheel_left.dae
- added link front_right_wheel, mass 0.4; collision cylinder length=0.0452 radius=0.0758; visual mesh filename=model://sentry_robot_visual/meshes/wheel_right.dae
- added link gimbal_yaw_link, mass 0.1; visual mesh filename=model://sentry_robot_visual/meshes/gimbal_pitch.dae; visual mesh filename=model://sentry_robot_visual/meshes/gimbal_yaw.dae
- added link rear_left_wheel, mass 0.4; collision cylinder length=0.0452 radius=0.0758; visual mesh filename=model://sentry_robot_visual/meshes/wheel_right.dae
- added link rear_right_wheel, mass 0.4; collision cylinder length=0.0452 radius=0.0758; visual mesh filename=model://sentry_robot_visual/meshes/wheel_left.dae
- added link sim_chassis_link, mass 50.0; collision box size=0.6 0.6 0.16; visual mesh filename=model://sentry_robot_visual/meshes/chassis_base.dae
Joints:
- added joint front_left_wheel_joint: type continuous, parent sim_chassis_link, child front_left_wheel, origin xyz=0.2242 0.2774 -0.2242 rpy=0 0 0, axis 0 1 0
- added joint front_right_wheel_joint: type continuous, parent sim_chassis_link, child front_right_wheel, origin xyz=0.2242 -0.2774 -0.2242 rpy=0 0 0, axis 0 1 0
- added joint gimbal_yaw_joint: type continuous, parent sim_chassis_link, child gimbal_yaw_link, origin xyz=0 0 0 rpy=0 0 0, axis 0 0 1
- added joint rear_left_wheel_joint: type continuous, parent sim_chassis_link, child rear_left_wheel, origin xyz=-0.2242 0.2774 -0.2242 rpy=0 0 0, axis 0 1 0
- added joint rear_right_wheel_joint: type continuous, parent sim_chassis_link, child rear_right_wheel, origin xyz=-0.2242 -0.2774 -0.2242 rpy=0 0 0, axis 0 1 0
